File: 12v-booster.kicad_pcb (KiCad board)
At the start: 2 copper layers, 21.9 x 10.3 mm, 18 parts, among them J1 Conn_01x04, J2 Conn_01x03, Q1 BSS214NW, U1 TPS55340-Q1

Commit message: Fixed solder mask clearance
Signed-off-by: Aaron Williams <aaron.w2@gmail.com>
Connections:
- net Net-(C5-Pad1) renamed /SS
- net Net-(C6-Pad1) renamed /COMP
- net Net-(R1-Pad2) renamed /FB
- net Net-(R2-Pad1) renamed /FREQ
Other:
- rule pad_to_mask_clearance: 0.0508 -> -0.0508
- board text added: "Version 1.2.2"
- board text removed: "Version 1.2.1"
