File: 12v-booster.sch (KiCad schematic (older format))
At the start: 18 parts, among them J1 Conn_01x04, J2 Conn_01x03, Q1 BSS214NW, U1 TPS55340-Q1

Commit message: Fixed solder mask clearance
Signed-off-by: Aaron Williams <aaron.w2@gmail.com>
Parts:
- C7: MFR Samsung -> Murata; MPN CL10B473KO8WPNC -> GRM188R61H474KA12D; SPN 1276-6852-1-ND -> 490-11994-1-ND
- U1: symbol texas:TPS55340-Q1 -> 12v-booster-rescue:TPS55340-Q1-texas
Connections:
- net labels added: COMP, FB, FREQ, SS
- no-connect marks 0 -> 1
Changed lines of the file:
@@
 $EndDescr
 $Comp
-L texas:TPS55340-Q1 U1
+L 12v-booster-rescue:TPS55340-Q1-texas U1
 U 1 1 5BAB0E99
 P 4950 3000
@@
 F 1 "47nF" H 6515 3555 50  0000 L CNN
 F 2 "Capacitor_SMD:C_0603_1608Metric" H 6438 3450 50  0001 C CNN
-F 3 "http://www.samsungsem.com/kr/support/product-search/mlcc/CL10B473KO8WPNC.jsp" H 6400 3600 50  0001 C CNN
-F 4 "Samsung" H 0   0   50  0001 C CNN "MFR"
-F 5 "CL10B473KO8WPNC" H 0   0   50  0001 C CNN "MPN"
-F 6 "Digikey" H 0   0   50  0001 C CNN "SPR"
-F 7 "1276-6852-1-ND" H 0   0   50  0001 C CNN "SPN"
+F 3 "" H 6400 3600 50  0001 C CNN
+F 4 "Murata" H 0   0   50  0001 C CNN "MFR"
+F 5 "GRM188R61H474KA12D" H 0   0   50  0001 C CNN "MPN"
+F 6 "Digikey" H 0   0   50  0001 C CNN "SPR"
+F 7 "490-11994-1-ND" H 0   0   50  0001 C CNN "SPN"
 F 8 "-" H 0   0   50  0001 C CNN "SPURL"
 	1    6400 3600
-	1    0    0    -1
-$EndComp
-$Comp
-L Device:R R4
-U 1 1 5BAB1556
-P 7100 3250
-F 0 "R4" H 7170 3296 50  0000 L CNN
-F 1 "10k" H 7170 3205 50  0000 L CNN
-F 2 "Resistor_SMD:R_0603_1608Metric" V 7030 3250 50  0001 C CNN
-F 3 "http://www.vishay.com/docs/20035/dcrcwe3.pdf" H 7100 3250 50  0001 C CNN
-F 4 "Vishay Dale" H 0   0   50  0001 C CNN "MFR"
-F 5 "CRCW060310K0FKEC" H 0   0   50  0001 C CNN "MPN"
-F 6 "Digikey" H 0   0   50  0001 C CNN "SPR"
-F 7 "541-2979-1-ND" H 0   0   50  0001 C CNN "SPN"
-F 8 "-" H 0   0   50  0001 C CNN "SPURL"
-	1    7100 3250
-	1    0    0    -1
-$EndComp
-$Comp
-L Device:R R1
-U 1 1 5BAB15CB
-P 7100 2600
-F 0 "R1" H 7170 2646 50  0000 L CNN
-F 1 "86.6k" H 7170 2555 50  0000 L CNN
-F 2 "Resistor_SMD:R_0603_1608Metric" V 7030 2600 50  0001 C CNN
-F 3 "http://www.vishay.com/docs/20035/dcrcwe3.pdf" H 7100 2600 50  0001 C CNN
-F 4 "Vishay Dale" H 0   0   50  0001 C CNN "MFR"
-F 5 "CRCW060386K6FKEA" H 0   0   50  0001 C CNN "MPN"
-F 6 "Digikey" H 0   0   50  0001 C CNN "SPR"
-F 7 "541-86.6KHCT-ND" H 0   0   50  0001 C CNN "SPN"
-F 8 "-" H 0   0   50  0001 C CNN "SPURL"
-	1    7100 2600
 	1    0    0    -1
 $EndComp
@@
 	5850 3750 6400 3750
 Wire Wire Line
-	7100 3100 7100 2750
-Wire Wire Line
 	5850 2750 7100 2750
 Wire Wire Line
-	7100 2450 6450 2450
-Wire Wire Line
 	5850 2550 5850 2450
 Wire Wire Line
@@
 	5850 2450 6150 2450
 Wire Wire Line
-	7100 2450 7550 2450
-Wire Wire Line
 	7550 2450 7550 2700
 Wire Wire Line
@@
 	8000 2450 8000 2700
 Wire Wire Line
-	6400 3750 7100 3750
-Wire Wire Line
-	7100 3750 7100 3400
-Wire Wire Line
-	7100 3750 7550 3750
-Wire Wire Line
 	7550 3750 7550 3000
 Wire Wire Line
@@
 	8000 2450 8500 2450
 Wire Wire Line
+	2200 3050 2350 3050
+Wire Wire Line
+	2350 3150 2200 3150
+Wire Wire Line
+	8400 3900 8400 2850
+Wire Wire Line
+	8100 4100 8050 4100
+Wire Wire Line
+	2200 4100 2200 3250
+Wire Wire Line
+	8050 4100 2200 4100
+Wire Wire Line
+	8400 4400 8400 4300
+Wire Wire Line
+	8050 4400 8400 4400
+Wire Wire Line
+	5050 4200 5050 3900
+Wire Wire Line
+	8000 3750 8300 3750
+Wire Wire Line
+	8300 2750 8300 3750
+Wire Wire Line
+	8400 2850 8500 2850
+Wire Wire Line
+	8500 2750 8300 2750
+Wire Wire Line
+	8500 2550 8500 2650
+Wire Wire Line
 	8500 2450 8500 2550
-Wire Wire Line
-	2200 3050 2350 3050
-Wire Wire Line
-	2350 3150 2200 3150
-Wire Wire Line
-	8400 3900 8400 2850
-Wire Wire Line
-	8100 4100 8050 4100
-Wire Wire Line
-	2200 4100 2200 3250
-Wire Wire Line
-	8050 4100 2200 4100
-Wire Wire Line
-	8400 4400 8400 4300
-Wire Wire Line
-	8050 4400 8400 4400
-Wire Wire Line
-	5050 4200 5050 3900
-Wire Wire Line
-	8000 3750 8300 3750
-Wire Wire Line
-	8400 2850 8500 2850
-Wire Wire Line
-	8500 2750 8300 2750
-Wire Wire Line
-	8300 2750 8300 3750
 Connection ~ 4050 2400
 Connection ~ 3200 2400
@@
 Connection ~ 3200 3900
 Connection ~ 5850 3000
-Connection ~ 7100 2750
 Connection ~ 5850 2450
-Connection ~ 7100 2450
 Connection ~ 7550 2450
 Connection ~ 6400 3750
-Connection ~ 7100 3750
 Connection ~ 7550 3750
 Connection ~ 8000 2450
@@
 Connection ~ 8400 4400
 Connection ~ 5050 3900
-Wire Wire Line
-	8500 2550 8500 2650
 Connection ~ 8500 2550
+Text Label 5850 2750 0    50   ~ 0
+FB
+Text Label 5850 3350 1    50   ~ 0
+COMP
+Text Label 3700 2800 0    50   ~ 0
+FREQ
+Text Label 3950 3400 0    50   ~ 0
+SS
+NoConn ~ 5500 3900
+Wire Wire Line
+	7100 3750 7550 3750
+Wire Wire Line
+	6400 3750 7100 3750
+Connection ~ 7100 3750
+Wire Wire Line
+	7100 3750 7100 3400
+Wire Wire Line
+	7100 3100 7100 2750
+$Comp
+L Device:R R4
+U 1 1 5BAB1556
+P 7100 3250
+F 0 "R4" H 7170 3296 50  0000 L CNN
+F 1 "10k" H 7170 3205 50  0000 L CNN
+F 2 "Resistor_SMD:R_0603_1608Metric" V 7030 3250 50  0001 C CNN
+F 3 "http://www.vishay.com/docs/20035/dcrcwe3.pdf" H 7100 3250 50  0001 C CNN
+F 4 "Vishay Dale" H 0   0   50  0001 C CNN "MFR"
+F 5 "CRCW060310K0FKEC" H 0   0   50  0001 C CNN "MPN"
+F 6 "Digikey" H 0   0   50  0001 C CNN "SPR"
+F 7 "541-2979-1-ND" H 0   0   50  0001 C CNN "SPN"
+F 8 "-" H 0   0   50  0001 C CNN "SPURL"
+	1    7100 3250
+	1    0    0    -1
+$EndComp
+Connection ~ 7100 2750
+Wire Wire Line
+	7100 2450 7550 2450
+Wire Wire Line
+	7100 2450 6450 2450
+Connection ~ 7100 2450
+$Comp
+L Device:R R1
+U 1 1 5BAB15CB
+P 7100 2600
+F 0 "R1" H 7170 2646 50  0000 L CNN
+F 1 "86.6k" H 7170 2555 50  0000 L CNN
+F 2 "Resistor_SMD:R_0603_1608Metric" V 7030 2600 50  0001 C CNN
+F 3 "http://www.vishay.com/docs/20035/dcrcwe3.pdf" H 7100 2600 50  0001 C CNN
+F 4 "Vishay Dale" H 0   0   50  0001 C CNN "MFR"
+F 5 "CRCW060386K6FKEA" H 0   0   50  0001 C CNN "MPN"
+F 6 "Digikey" H 0   0   50  0001 C CNN "SPR"
+F 7 "541-86.6KHCT-ND" H 0   0   50  0001 C CNN "SPN"
+F 8 "-" H 0   0   50  0001 C CNN "SPURL"
+	1    7100 2600
+	1    0    0    -1
+$EndComp
 $EndSCHEMATC
